Commit message: Adjust motor direction, distance (inaccurate).

File: urdf/snake_stl.urdf (robot description, URDF)
Before this commit: robot test_robot, 21 links, 20 joints
Links:
- added link bracket_011, mass 0.0060293114415; collision mesh filename=package://snake/mesh/xh430_frame.stl; visual mesh filename=package://snake/mesh/xh430_frame.stl
- added link bracket_012, mass 0.0060293114415; collision mesh filename=package://snake/mesh/xh430_frame.stl; visual mesh filename=package://snake/mesh/xh430_frame.stl
- added link bracket_013, mass 0.0060293114415; collision mesh filename=package://snake/mesh/xh430_frame.stl; visual mesh filename=package://snake/mesh/xh430_frame.stl
- added link bracket_014, mass 0.0060293114415; collision mesh filename=package://snake/mesh/xh430_frame.stl; visual mesh filename=package://snake/mesh/xh430_frame.stl
- added link bracket_015, mass 0.0060293114415; collision mesh filename=package://snake/mesh/xh430_frame.stl; visual mesh filename=package://snake/mesh/xh430_frame.stl
- added link bracket_016, mass 0.0060293114415; collision mesh filename=package://snake/mesh/xh430_frame.stl; visual mesh filename=package://snake/mesh/xh430_frame.stl
- added link bracket_017, mass 0.0060293114415; collision mesh filename=package://snake/mesh/xh430_frame.stl; visual mesh filename=package://snake/mesh/xh430_frame.stl
- added link bracket_018, mass 0.0060293114415; collision mesh filename=package://snake/mesh/xh430_frame.stl; visual mesh filename=package://snake/mesh/xh430_frame.stl
- added link bracket_019, mass 0.0060293114415; collision mesh filename=package://snake/mesh/xh430_frame.stl; visual mesh filename=package://snake/mesh/xh430_frame.stl
- added link bracket_020, mass 0.0060293114415; collision mesh filename=package://snake/mesh/xh430_frame.stl; visual mesh filename=package://snake/mesh/xh430_frame.stl
- added link bracket_021, mass 0.0060293114415; collision mesh filename=package://snake/mesh/xh430_frame.stl; visual mesh filename=package://snake/mesh/xh430_frame.stl
- added link bracket_022, mass 0.0060293114415; collision mesh filename=package://snake/mesh/xh430_frame.stl; visual mesh filename=package://snake/mesh/xh430_frame.stl
- added link bracket_023, mass 0.0060293114415; collision mesh filename=package://snake/mesh/xh430_frame.stl; visual mesh filename=package://snake/mesh/xh430_frame.stl
- added link bracket_024, mass 0.0060293114415; collision mesh filename=package://snake/mesh/xh430_frame.stl; visual mesh filename=package://snake/mesh/xh430_frame.stl
- added link dynamixel_006, mass 0.082; collision mesh filename=package://snake/mesh/XH_430_idler.stl; visual mesh filename=package://snake/mesh/XH_430_idler.stl
- added link dynamixel_007, mass 0.082; collision mesh filename=package://snake/mesh/XH_430_idler.stl; visual mesh filename=package://snake/mesh/XH_430_idler.stl
- added link dynamixel_008, mass 0.082; collision mesh filename=package://snake/mesh/XH_430_idler.stl; visual mesh filename=package://snake/mesh/XH_430_idler.stl
- added link dynamixel_009, mass 0.082; collision mesh filename=package://snake/mesh/XH_430_idler.stl; visual mesh filename=package://snake/mesh/XH_430_idler.stl
- added link dynamixel_010, mass 0.082; collision mesh filename=package://snake/mesh/XH_430_idler.stl; visual mesh filename=package://snake/mesh/XH_430_idler.stl
- added link dynamixel_011, mass 0.082; collision mesh filename=package://snake/mesh/XH_430_idler.stl; visual mesh filename=package://snake/mesh/XH_430_idler.stl
- added link dynamixel_012, mass 0.082; collision mesh filename=package://snake/mesh/XH_430_idler.stl; visual mesh filename=package://snake/mesh/XH_430_idler.stl
- added link dynamixel_106, mass 0.082; collision mesh filename=package://snake/mesh/XH_430_idler.stl; visual mesh filename=package://snake/mesh/XH_430_idler.stl
- added link dynamixel_107, mass 0.082; collision mesh filename=package://snake/mesh/XH_430_idler.stl; visual mesh filename=package://snake/mesh/XH_430_idler.stl
- added link dynamixel_108, mass 0.082; collision mesh filename=package://snake/mesh/XH_430_idler.stl; visual mesh filename=package://snake/mesh/XH_430_idler.stl
- added link dynamixel_109, mass 0.082; collision mesh filename=package://snake/mesh/XH_430_idler.stl; visual mesh filename=package://snake/mesh/XH_430_idler.stl
- added link dynamixel_110, mass 0.082; collision mesh filename=package://snake/mesh/XH_430_idler.stl; visual mesh filename=package://snake/mesh/XH_430_idler.stl
- added link dynamixel_111, mass 0.082; collision mesh filename=package://snake/mesh/XH_430_idler.stl; visual mesh filename=package://snake/mesh/XH_430_idler.stl
- added link dynamixel_112, mass 0.082; collision mesh filename=package://snake/mesh/XH_430_idler.stl; visual mesh filename=package://snake/mesh/XH_430_idler.stl
- link bracket_001: geometry collision mesh filename=package://snake/mesh/xh430_frame.stl; visual mesh filename=package://snake/mesh/xh430_frame.stl
- link bracket_002: geometry collision mesh filename=package://snake/mesh/xh430_frame.stl; visual mesh filename=package://snake/mesh/xh430_frame.stl
- link bracket_003: geometry collision mesh filename=package://snake/mesh/xh430_frame.stl; visual mesh filename=package://snake/mesh/xh430_frame.stl
- link bracket_004: geometry collision mesh filename=package://snake/mesh/xh430_frame.stl; visual mesh filename=package://snake/mesh/xh430_frame.stl
- link bracket_005: geometry collision mesh filename=package://snake/mesh/xh430_frame.stl; visual mesh filename=package://snake/mesh/xh430_frame.stl
- link bracket_006: geometry collision mesh filename=package://snake/mesh/xh430_frame.stl; visual mesh filename=package://snake/mesh/xh430_frame.stl
- link bracket_007: geometry collision mesh filename=package://snake/mesh/xh430_frame.stl; visual mesh filename=package://snake/mesh/xh430_frame.stl
- link bracket_008: geometry collision mesh filename=package://snake/mesh/xh430_frame.stl; visual mesh filename=package://snake/mesh/xh430_frame.stl
- link bracket_009: geometry collision mesh filename=package://snake/mesh/xh430_frame.stl; visual mesh filename=package://snake/mesh/xh430_frame.stl
- link bracket_010: geometry collision mesh filename=package://snake/mesh/xh430_frame.stl; visual mesh filename=package://snake/mesh/xh430_frame.stl
- link dynamixel_001: mass 0.023967239474 -> 0.082; geometry collision mesh filename=package://snake/mesh/XH_430_idler.stl; visual mesh filename=package://snake/mesh/XH_430_idler.stl
- link dynamixel_002: mass 0.023967239474 -> 0.082; geometry collision mesh filename=package://snake/mesh/XH_430_idler.stl; visual mesh filename=package://snake/mesh/XH_430_idler.stl
- link dynamixel_003: mass 0.023967239474 -> 0.082; geometry collision mesh filename=package://snake/mesh/XH_430_idler.stl; visual mesh filename=package://snake/mesh/XH_430_idler.stl
- link dynamixel_004: mass 0.023967239474 -> 0.082; geometry collision mesh filename=package://snake/mesh/XH_430_idler.stl; visual mesh filename=package://snake/mesh/XH_430_idler.stl
- link dynamixel_005: mass 0.023967239474 -> 0.082; geometry collision mesh filename=package://snake/mesh/XH_430_idler.stl; visual mesh filename=package://snake/mesh/XH_430_idler.stl
- link dynamixel_101: mass 0.023967239474 -> 0.082; geometry collision mesh filename=package://snake/mesh/XH_430_idler.stl; visual mesh filename=package://snake/mesh/XH_430_idler.stl
- link dynamixel_102: mass 0.023967239474 -> 0.082; geometry collision mesh filename=package://snake/mesh/XH_430_idler.stl; visual mesh filename=package://snake/mesh/XH_430_idler.stl
- link dynamixel_103: mass 0.023967239474 -> 0.082; geometry collision mesh filename=package://snake/mesh/XH_430_idler.stl; visual mesh filename=package://snake/mesh/XH_430_idler.stl
- link dynamixel_104: mass 0.023967239474 -> 0.082; geometry collision mesh filename=package://snake/mesh/XH_430_idler.stl; visual mesh filename=package://snake/mesh/XH_430_idler.stl
- link dynamixel_105: mass 0.023967239474 -> 0.082; geometry collision mesh filename=package://snake/mesh/XH_430_idler.stl; visual mesh filename=package://snake/mesh/XH_430_idler.stl
Joints:
- added joint fixed_010: type fixed, parent bracket_010, child dynamixel_006, origin xyz=0.0605 0 0 rpy=-1.57079632679 0 0, limit lower=-1.57079632679 upper=1.57079632679 effort=0 velocity=0
- added joint fixed_011: type fixed, parent bracket_011, child dynamixel_106, origin xyz=0.0605 0 0 rpy=1.57079632679 0 0, limit lower=-1.57079632679 upper=1.57079632679 effort=0 velocity=0
- added joint fixed_012: type fixed, parent bracket_012, child dynamixel_007, origin xyz=0.0605 0 0 rpy=-1.57079632679 0 0, limit lower=-1.57079632679 upper=1.57079632679 effort=0 velocity=0
- added joint fixed_013: type fixed, parent bracket_013, child dynamixel_107, origin xyz=0.0605 0 0 rpy=1.57079632679 0 0, limit lower=-1.57079632679 upper=1.57079632679 effort=0 velocity=0
- added joint fixed_014: type fixed, parent bracket_014, child dynamixel_008, origin xyz=0.0605 0 0 rpy=-1.57079632679 0 0, limit lower=-1.57079632679 upper=1.57079632679 effort=0 velocity=0
- added joint fixed_015: type fixed, parent bracket_015, child dynamixel_108, origin xyz=0.0605 0 0 rpy=1.57079632679 0 0, limit lower=-1.57079632679 upper=1.57079632679 effort=0 velocity=0
- added joint fixed_016: type fixed, parent bracket_016, child dynamixel_009, origin xyz=0.0605 0 0 rpy=-1.57079632679 0 0, limit lower=-1.57079632679 upper=1.57079632679 effort=0 velocity=0
- added joint fixed_017: type fixed, parent bracket_017, child dynamixel_109, origin xyz=0.0605 0 0 rpy=1.57079632679 0 0, limit lower=-1.57079632679 upper=1.57079632679 effort=0 velocity=0
- added joint fixed_018: type fixed, parent bracket_018, child dynamixel_010, origin xyz=0.0605 0 0 rpy=-1.57079632679 0 0, limit lower=-1.57079632679 upper=1.57079632679 effort=0 velocity=0
- added joint fixed_019: type fixed, parent bracket_019, child dynamixel_110, origin xyz=0.0605 0 0 rpy=1.57079632679 0 0, limit lower=-1.57079632679 upper=1.57079632679 effort=0 velocity=0
- added joint fixed_020: type fixed, parent bracket_020, child dynamixel_011, origin xyz=0.0605 0 0 rpy=-1.57079632679 0 0, limit lower=-1.57079632679 upper=1.57079632679 effort=0 velocity=0
- added joint fixed_021: type fixed, parent bracket_021, child dynamixel_111, origin xyz=0.0605 0 0 rpy=1.57079632679 0 0, limit lower=-1.57079632679 upper=1.57079632679 effort=0 velocity=0
- added joint fixed_022: type fixed, parent bracket_022, child dynamixel_012, origin xyz=0.0605 0 0 rpy=-1.57079632679 0 0, limit lower=-1.57079632679 upper=1.57079632679 effort=0 velocity=0
- added joint fixed_023: type fixed, parent bracket_023, child dynamixel_112, origin xyz=0.0605 0 0 rpy=1.57079632679 0 0, limit lower=-1.57079632679 upper=1.57079632679 effort=0 velocity=0
- added joint joint_011: type revolute, parent dynamixel_006, child bracket_011, origin xyz=0 0 0 rpy=0 0 0, axis 0 1 0, limit lower=-1.57079632679 upper=1.57079632679 effort=0 velocity=0
- added joint joint_012: type revolute, parent dynamixel_106, child bracket_012, origin xyz=0 0 0 rpy=0 0 0, axis 0 1 0, limit lower=-1.57079632679 upper=1.57079632679 effort=0 velocity=0
- added joint joint_013: type revolute, parent dynamixel_007, child bracket_013, origin xyz=0 0 0 rpy=0 0 0, axis 0 1 0, limit lower=-1.57079632679 upper=1.57079632679 effort=0 velocity=0
- added joint joint_014: type revolute, parent dynamixel_107, child bracket_014, origin xyz=0 0 0 rpy=0 0 0, axis 0 1 0, limit lower=-1.57079632679 upper=1.57079632679 effort=0 velocity=0
- added joint joint_015: type revolute, parent dynamixel_008, child bracket_015, origin xyz=0 0 0 rpy=0 0 0, axis 0 1 0, limit lower=-1.57079632679 upper=1.57079632679 effort=0 velocity=0
- added joint joint_016: type revolute, parent dynamixel_108, child bracket_016, origin xyz=0 0 0 rpy=0 0 0, axis 0 1 0, limit lower=-1.57079632679 upper=1.57079632679 effort=0 velocity=0
- added joint joint_017: type revolute, parent dynamixel_009, child bracket_017, origin xyz=0 0 0 rpy=0 0 0, axis 0 1 0, limit lower=-1.57079632679 upper=1.57079632679 effort=0 velocity=0
- added joint joint_018: type revolute, parent dynamixel_109, child bracket_018, origin xyz=0 0 0 rpy=0 0 0, axis 0 1 0, limit lower=-1.57079632679 upper=1.57079632679 effort=0 velocity=0
- added joint joint_019: type revolute, parent dynamixel_010, child bracket_019, origin xyz=0 0 0 rpy=0 0 0, axis 0 1 0, limit lower=-1.57079632679 upper=1.57079632679 effort=0 velocity=0
- added joint joint_020: type revolute, parent dynamixel_110, child bracket_020, origin xyz=0 0 0 rpy=0 0 0, axis 0 1 0, limit lower=-1.57079632679 upper=1.57079632679 effort=0 velocity=0
- added joint joint_021: type revolute, parent dynamixel_011, child bracket_021, origin xyz=0 0 0 rpy=0 0 0, axis 0 1 0, limit lower=-1.57079632679 upper=1.57079632679 effort=0 velocity=0
- added joint joint_022: type revolute, parent dynamixel_111, child bracket_022, origin xyz=0 0 0 rpy=0 0 0, axis 0 1 0, limit lower=-1.57079632679 upper=1.57079632679 effort=0 velocity=0
- added joint joint_023: type revolute, parent dynamixel_012, child bracket_023, origin xyz=0 0 0 rpy=0 0 0, axis 0 1 0, limit lower=-1.57079632679 upper=1.57079632679 effort=0 velocity=0
- added joint joint_024: type revolute, parent dynamixel_112, child bracket_024, origin xyz=0 0 0 rpy=0 0 0, axis 0 1 0, limit lower=-1.57079632679 upper=1.57079632679 effort=0 velocity=0
- joint fixed_001: origin xyz=0.046 0 0 rpy=1.57079632679 0 0 -> xyz=0.0605 0 0 rpy=1.57079632679 0 0
- joint fixed_002: origin xyz=0.046 0 0 rpy=-1.57079632679 0 0 -> xyz=0.0605 0 0 rpy=-1.57079632679 0 0
- joint fixed_003: origin xyz=0.046 0 0 rpy=1.57079632679 0 0 -> xyz=0.0605 0 0 rpy=1.57079632679 0 0
- joint fixed_004: origin xyz=0.046 0 0 rpy=-1.57079632679 0 0 -> xyz=0.0605 0 0 rpy=-1.57079632679 0 0
- joint fixed_005: origin xyz=0.046 0 0 rpy=1.57079632679 0 0 -> xyz=0.0605 0 0 rpy=1.57079632679 0 0
- joint fixed_006: origin xyz=0.046 0 0 rpy=-1.57079632679 0 0 -> xyz=0.0605 0 0 rpy=-1.57079632679 0 0
- joint fixed_007: origin xyz=0.046 0 0 rpy=1.57079632679 0 0 -> xyz=0.0605 0 0 rpy=1.57079632679 0 0
- joint fixed_008: origin xyz=0.046 0 0 rpy=-1.57079632679 0 0 -> xyz=0.0605 0 0 rpy=-1.57079632679 0 0
- joint fixed_009: origin xyz=0.046 0 0 rpy=1.57079632679 0 0 -> xyz=0.0605 0 0 rpy=1.57079632679 0 0

File: urdf/snake_stl.xacro (robot description, xacro)
@@ -17,5 +17,5 @@
   <xacro:property name="iyy_a" value="0"/>
   <xacro:property name="izz_a" value="0" />
-  <xacro:property name="fixed_pos" value="0.046" />
+  <xacro:property name="fixed_pos" value="0.0605" />
   <!-- 定義するdynamixelの名前 -->
   <xacro:property name="dynamixel_names" value="${[
@@ -192,5 +192,5 @@
             <color rgba="0.0 1.0 1.0 1.0"/>
           </material>
-                <origin rpy="0 0 0" xyz="0 0 0"/>
+                <origin rpy="${pi} ${pi/2} ${pi/2}" xyz="0 0 0"/>
         </visual>
         <!--物理的特性-->
@@ -224,5 +224,5 @@
           <color rgba="0.75 0.75 0.75 1"/>
         </material>
-              <origin rpy="0 0 0" xyz="0 0 0"/>
+              <origin rpy="${-pi/2} ${-pi/2} ${pi}" xyz="0.023 0 0"/>
       </visual>
       <!--物理的特性-->
@@ -266,5 +266,5 @@
       <xacro:if value="${'joint' in name}">
         <xacro:property name="joint_type" value="revolute"/>
-        <xacro:property name="x" value="${0}"/>
+        <xacro:property name="x" value="0"/>
         <xacro:property name="rpy" value="0 0 0"/>
       </xacro:if>
